File: RD16-Amplifier.sch (KiCad schematic (older format))
At the start: 45 parts, among them J1 RF_OUT, J2 RF_IN, J3 LPF_IN, J4 LPF_OUT, J5 13.8V Input, J6 PTT, J7 Conn_01x02, J8 Conn_01x02, K1 G5V-2, Q1 2N3906-SMD, Q2 IRF530, Q3 IRF530, T1 BN-43-202 1T:2T, U1 L7805

Commit message: gg
Parts:
- Q2, Q3: footprint Xenir:TO-220-Horizontal -> xenir:TO-220-Horizontal-RD-Mosfet
- T2: renamed from T?; footprint (none) -> xenir:T50_Transformer
- T3: renamed from T?; value T37_XFRM -> Ferrite Tube; footprint (none) -> xenir:Ferrite-Tube-Transformer-SMD
- gave numbers to parts that had none: 1
Changed lines of the file:
@@
 F 0 "Q2" H 5950 4100 50  0000 L CNN
 F 1 "IRF530" H 5550 4100 50  0000 L CNN
-F 2 "Xenir:TO-220-Horizontal" H 6050 3875 50  0001 L CIN
+F 2 "xenir:TO-220-Horizontal-RD-Mosfet" H 6050 3875 50  0001 L CIN
 F 3 "http://www.irf.com/product-info/datasheets/data/irf540n.pdf" H 5800 3950 50  0001 L CNN
 	1    5800 3950
@@
 F 0 "Q3" H 5950 5100 50  0000 L CNN
 F 1 "IRF530" H 5550 5100 50  0000 L CNN
-F 2 "Xenir:TO-220-Horizontal" H 6050 4875 50  0001 L CIN
+F 2 "xenir:TO-220-Horizontal-RD-Mosfet" H 6050 4875 50  0001 L CIN
 F 3 "http://www.irf.com/product-info/datasheets/data/irf540n.pdf" H 5800 4950 50  0001 L CNN
 	1    5800 4950
@@
 Connection ~ 4300 4350
 $Comp
-L xenir:T37_XFRM T?
+L xenir:T37_XFRM T3
 U 1 1 630FAECC
 P 8500 4000
-F 0 "T?" H 8500 4041 50  0000 C CNN
-F 1 "T37_XFRM" H 8500 3950 50  0000 C CNN
-F 2 "" H 8500 4000 50  0001 C CNN
+F 0 "T3" H 8500 4041 50  0000 C CNN
+F 1 "Ferrite Tube" H 8500 3950 50  0000 C CNN
+F 2 "xenir:Ferrite-Tube-Transformer-SMD" H 8500 4000 50  0001 C CNN
 F 3 "" H 8500 4000 50  0001 C CNN
 	1    8500 4000
@@
 	6300 4325 6300 4550
 $Comp
-L xenir:T37_XFRM T?
+L xenir:T37_XFRM T2
 U 1 1 63134E4D
 P 7250 4000
-F 0 "T?" H 7250 4041 50  0000 C CNN
+F 0 "T2" H 7250 4041 50  0000 C CNN
 F 1 "T50-43" H 7250 3950 50  0000 C CNN
-F 2 "" H 7250 4000 50  0001 C CNN
+F 2 "xenir:T50_Transformer" H 7250 4000 50  0001 C CNN
 F 3 "" H 7250 4000 50  0001 C CNN
 	1    7250 4000
@@
 Connection ~ 6850 5700
 $Comp
-L xenir:Capacitor C?
+L xenir:Capacitor C9
 U 1 1 63196FB6
 P 7800 4900
-F 0 "C?" V 7771 5015 28  0000 L CNN
+F 0 "C9" V 7771 5015 28  0000 L CNN
 F 1 ".1uF" V 7828 5015 28  0000 L CNN
 F 2 "Xenir:Capacitor 1206" H 7800 4750 50  0001 C CNN
@@
 $EndComp
 $Comp
-L power:GND #PWR?
+L power:GND #PWR0103
 U 1 1 63196FC0
 P 7800 5050
-F 0 "#PWR?" H 7800 4800 50  0001 C CNN
+F 0 "#PWR0103" H 7800 4800 50  0001 C CNN
 F 1 "GND" H 7805 4877 50  0000 C CNN
 F 2 "" H 7800 5050 50  0001 C CNN

Commit message: more fixes
Parts:
- added C?: 33pF, Xenir:Capacitor 1206, symbol xenir:Capacitor
- added D8, D9: 1N914, Diode_SMD:D_SOD-123, symbol Diode:1N914
Connections:
- net Q2Drain: now also C?.1
- net Q3Drain: now also C?.2
- net at D6.1 (K): now also D8.2 (A); no longer D7.2 (A)
- new net: D7.2 (A), D9.1 (K)
- new net: D8.1 (K), D9.2 (A)
Changed lines of the file:
@@
 	1    0    0    -1
 $EndComp
-Wire Wire Line
-	10000 2450 10000 2750
 $Comp
 L Connector_Generic:Conn_01x02 J7
@@
 $EndComp
 Connection ~ 7800 4750
+$Comp
+L Diode:1N914 D8
+U 1 1 6308F48C
+P 10150 2450
+F 0 "D8" H 10150 2233 50  0000 C CNN
+F 1 "1N914" H 10150 2324 50  0000 C CNN
+F 2 "Diode_SMD:D_SOD-123" H 10150 2275 50  0001 C CNN
+F 3 "http://www.vishay.com/docs/85622/1n914.pdf" H 10150 2450 50  0001 C CNN
+	1    10150 2450
+	-1   0    0    1
+$EndComp
+$Comp
+L Diode:1N914 D9
+U 1 1 6308F496
+P 10150 2750
+F 0 "D9" H 10150 2967 50  0000 C CNN
+F 1 "1N914" H 10150 2876 50  0000 C CNN
+F 2 "Diode_SMD:D_SOD-123" H 10150 2575 50  0001 C CNN
+F 3 "http://www.vishay.com/docs/85622/1n914.pdf" H 10150 2750 50  0001 C CNN
+	1    10150 2750
+	1    0    0    -1
+$EndComp
+Wire Wire Line
+	10300 2450 10450 2450
+Wire Wire Line
+	10450 2450 10450 2750
+Wire Wire Line
+	10450 2750 10300 2750
+$Comp
+L xenir:Capacitor C?
+U 1 1 630B2858
+P 8100 4450
+F 0 "C?" V 8050 4250 28  0000 L CNN
+F 1 "33pF" V 8100 4250 28  0000 L CNN
+F 2 "Xenir:Capacitor 1206" H 8100 4300 50  0001 C CNN
+F 3 "" H 8100 4300 50  0001 C CNN
+	1    8100 4450
+	0    1    1    0
+$EndComp
+Wire Wire Line
+	8100 4150 8100 4300
+Connection ~ 8100 4150
+Wire Wire Line
+	8100 4600 8100 4750
+Connection ~ 8100 4750
 $EndSCHEMATC
